File: pcb/projekt.brd (EAGLE design)
At the start: 12 parts

Commit message: pcb change 	modified:   pcb/projekt.brd
Parts:
- E$10, E$11, E$12, E$9: device pinhead:1X05 -> pinhead:1X08
- moved E$10 30.7 mm to (88.9, 38.1)
- moved E$9 30.7 mm to (76.2, 38.1)
- moved E$3 30.5 mm to (34.3, 38.1)
- moved E$4 14.4 mm to (61.0, 15.2)
- moved E$11 8.03 mm to (45.7, 48.3)
- moved E$12 8.03 mm to (58.4, 48.3)
Other:
- board text added: "pa1-0 pa3-2 pa5-4 pa7-6 pb1-0 pb10-2 pb11-12 pb13-14 pb15-pa8 tx-rx"
- board text added: "pd-nst pc15-pd0 pc13-pc14 pb5-vbat bt0-pb8 pb6-pb7 pb4-pb5 pa15-pb3 pa13-pa14 pa11-pa12"
- board text added: "vmt gnd 2b 2a 1a 1b vdd gnd"
- board text added: "~en ms1 ms2 ms3 ~rs ~sl stp dir"
Changed lines of the file:
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@@
 <text x="29.845" y="32.385" size="1.778" layer="1" rot="R180">3,3</text>
 <text x="40.005" y="32.385" size="1.778" layer="1" rot="R180">3,3</text>
-<text x="25.4" y="20.32" size="1.778" layer="1">vbat</text>
-<text x="-2.54" y="40.64" size="1.778" layer="1">5v</text>
-<text x="-0.635" y="40.005" size="1.778" layer="1" rot="R180">tx</text>
-<text x="0" y="38.1" size="1.778" layer="1" rot="R180">rx</text>
-<text x="0" y="34.925" size="1.778" layer="1" rot="R180">gnd</text>
+<text x="8.255" y="20.955" size="1.778" layer="1">vbat</text>
+<text x="29.21" y="41.275" size="1.778" layer="1">5v</text>
+<text x="31.115" y="40.005" size="1.778" layer="1" rot="R180">tx</text>
+<text x="31.115" y="37.465" size="1.778" layer="1" rot="R180">rx</text>
+<text x="31.115" y="34.925" size="1.778" layer="1" rot="R180">gnd</text>
+<text x="43.18" y="58.42" size="1.778" layer="1" rot="R180">~en
+ms1
+ms2
+ms3
+~rs
+~sl
+stp
+dir</text>
+<text x="66.04" y="58.42" size="1.778" layer="1" rot="R180">vmt
+gnd
+2b
+2a
+1a
+1b
+vdd
+gnd</text>
+<text x="73.66" y="48.26" size="1.778" layer="1" rot="R180">~en
+ms1
+ms2
+ms3
+~rs
+~sl
+stp
+dir</text>
+<text x="96.52" y="48.26" size="1.778" layer="1" rot="R180">vmt
+gnd
+2b
+2a
+1a
+1b
+vdd
+gnd</text>
+<text x="36.195" y="5.715" size="1.6764" layer="1">pa1-0
+pa3-2
+pa5-4
+pa7-6
+pb1-0
+pb10-2
+pb11-12
+pb13-14
+pb15-pa8
+tx-rx</text>
+<text x="-10.16" y="5.08" size="1.6764" layer="1">pd-nst
+pc15-pd0
+pc13-pc14
+pb5-vbat
+bt0-pb8
+pb6-pb7
+pb4-pb5
+pa15-pb3
+pa13-pa14
+pa11-pa12</text>
 </plain>
 <attributes>
@@
 <element name="E$2" library="pinhead" package="2X12" value="" x="33.02" y="17.78" rot="R270"/>
 <element name="E$1" library="pinhead" package="2X12" value="" x="5.08" y="17.78" rot="R270"/>
-<element name="E$3" library="pinhead" package="1X04" value="" x="3.81" y="38.1" rot="R90"/>
-<element name="E$4" library="con-wago-500" package="W237-4" value="" x="50.8" y="5.08"/>
+<element name="E$3" library="pinhead" package="1X04" value="" x="34.29" y="38.1" rot="R90"/>
+<element name="E$4" library="con-wago-500" package="W237-4" value="" x="60.96" y="15.24"/>
 <element name="E$5" library="con-wago-500" package="W237-4" value="" x="73.66" y="5.08"/>
 <element name="E$6" library="con-wago-500" package="W237-4" value="" x="10.16" y="60.96"/>
 <element name="E$7" library="con-wago-500" package="W237-4" value="" x="86.36" y="15.24"/>
 <element name="E$8" library="con-wago-500" package="W237-4" value="" x="15.24" y="78.74"/>
-<element name="E$9" library="pinhead" package="1X05" value="" x="48.26" y="25.4" rot="R90"/>
-<element name="E$10" library="pinhead" package="1X05" value="" x="60.96" y="25.4" rot="R90"/>
-<element name="E$11" library="pinhead" package="1X05" value="" x="48.26" y="40.64" smashed="yes" rot="R90">
-<attribute name="NAME" x="46.4312" y="34.2138" size="1.27" layer="25" ratio="10" rot="R90"/>
-<attribute name="VALUE" x="51.435" y="34.29" size="1.27" layer="27" rot="R90"/>
-</element>
-<element name="E$12" library="pinhead" package="1X05" value="" x="60.96" y="40.64" rot="R90"/>
+<element name="E$9" library="pinhead" package="1X08" value="" x="76.2" y="38.1" rot="R90"/>
+<element name="E$10" library="pinhead" package="1X08" value="" x="88.9" y="38.1" rot="R90"/>
+<element name="E$11" library="pinhead" package="1X08" value="" x="45.72" y="48.26" rot="R90"/>
+<element name="E$12" library="pinhead" package="1X08" value="" x="58.42" y="48.26" rot="R90"/>
 </elements>
 <signals>
@@
 </board>
 </drawing>
+<compatibility>
+<note version="6.3" minversion="6.2.2" severity="warning">
+Since Version 6.2.2 text objects can contain more than one line,
+which will not be processed correctly with this version.
+</note>
+</compatibility>
 </eagle>

Commit message: 'pcb_script'
Parts:
- added E$13: (no value), con-wago-500:W237-103
- added E$14, E$15: (no value), con-wago-500:W237-102
- moved E$5 65.3 mm to (58.4, 68.6)
- moved E$4 35.3 mm to (91.4, 33.0), turned to 90 degrees
- moved E$10 32.5 mm to (68.6, 12.7)
- moved E$9 32.5 mm to (55.9, 12.7)
- moved E$6 25.5 mm to (35.6, 58.4)
- moved E$8 22.7 mm to (35.6, 68.6)
- moved E$11 14.4 mm to (55.9, 38.1)
- moved E$12 14.4 mm to (68.6, 38.1)
- moved E$7 7.18 mm to (91.4, 10.2), turned to 90 degrees
- moved E$2 3.59 mm to (30.5, 15.2)
- moved E$1 3.59 mm to (2.54, 15.2)
- moved E$3 3.59 mm to (31.8, 35.6)
Connections:
- new net S$1: E$1.23, E$1.24, E$15.2, E$2.23, E$2.24
- new net S$2: E$12.1, E$12.7
- new net S$5: E$10.1, E$10.7
Routing:
- net S$1: track 0.00 -> 197.3 mm

Commit message: 'pcb_rotate'
Parts:
- added E$16: (no value), con-wago-500:W237-102
- moved E$6 30.6 mm to (5.08, 61.0), turned to 270 degrees
- moved E$3 26.7 mm to (5.08, 34.3), turned to 180 degrees
- moved E$1 25.0 mm to (25.4, 5.08), turned to 0 degrees
- moved E$5 25.0 mm to (81.3, 78.7), turned to 180 degrees
- moved E$8 25.0 mm to (58.4, 78.7), turned to 180 degrees
- moved E$2 18.5 mm to (25.4, 33.0), turned to 0 degrees
- moved E$15 10.2 mm to (5.08, 78.7)
- moved E$7 5.68 mm to (86.4, 7.62)
- moved E$13 5.08 mm to (86.4, 66.0)
- moved E$14 5.08 mm to (86.4, 50.8)
- moved E$4 5.08 mm to (86.4, 33.0)
Connections:
- new net S$10: E$1.9, E$11.2
- new net S$11: E$11.8, E$2.16
- new net S$12: E$13.1, E$2.10
- new net S$13: E$13.3, E$2.9
- new net S$14: E$1.10, E$16.2
- new net S$15: E$10.8, E$12.8, E$15.1
- new net S$16: E$1.1, E$1.2, E$10.2, E$12.2
- new net S$17: E$11.4, E$2.18, E$9.4
- new net S$18: E$1.12, E$11.1
- new net S$19: E$13.2, E$2.7
- new net S$20: E$2.13, E$9.1
- new net S$21: E$2.15, E$9.2
- new net S$22: E$2.17, E$9.8
- new net S$23: E$14.2, E$3.4
- new net S$24: E$1.23, E$1.24, E$10.1, E$10.7, E$12.1
- new net S$3: E$10.4, E$7.2
- new net S$4: E$10.5, E$7.3
- new net S$6: E$12.3, E$4.1
- new net S$7: E$12.4, E$4.2
- new net S$8: E$12.5, E$4.3
- new net S$9: E$12.6, E$4.4
- net S$1: now also E$12.7, E$14.1, E$16.1; no longer E$1.23, E$1.24, E$2.23, E$2.24
- net S$2: now also E$10.3, E$7.1; no longer E$12.1, E$12.7
- net S$5: now also E$10.6, E$7.4; no longer E$10.1, E$10.7
Routing:
- net S$15: track 0.00 -> 202.6 mm
- net S$1: track 197.3 -> 41.1 mm
- net S$13: track 0.00 -> 154.7 mm
- net S$19: track 0.00 -> 137.7 mm
- net S$23: track 0.00 -> 119.1 mm
- net S$16: track 0.00 -> 106.0 mm
- net S$24: track 0.00 -> 86.0 mm
- net S$12: track 0.00 -> 80.1 mm
- net S$10: track 0.00 -> 77.9 mm
- net S$18: track 0.00 -> 73.6 mm
- net S$17: track 0.00 -> 67.9 mm
- net S$20: track 0.00 -> 54.7 mm
- net S$21: track 0.00 -> 50.2 mm
- net S$11: track 0.00 -> 34.2 mm
- net S$22: track 0.00 -> 33.5 mm
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Other:
- board text added: "pd-nst pc15-pd0 pc13-pc14 pb9-vbat bt0-pb8 pb6-pb7 pb4-pb5 pa15-pb3 pa13-pa14 pa11-pa12"
- board text removed: "pd-nst pc15-pd0 pc13-pc14 pb5-vbat bt0-pb8 pb6-pb7 pb4-pb5 pa15-pb3 pa13-pa14 pa11-pa12"

Commit message: modified:   pcb/projekt.brd 	modified:   pcb/readme.scr
Parts:
- removed E$6: (no value), con-wago-500:W237-4
- E$5: device con-wago-500:W237-4 -> con-wago-500:W237-102
- moved E$8 15.3 mm to (43.2, 78.1)
- moved E$5 5.12 mm to (86.4, 78.1)
- moved E$16 2.62 mm to (20.3, 78.1), turned to 270 degrees
- moved E$15 0.90 mm to (4.45, 78.1)
Connections:
- net S$15 renamed +12V
- removed net S$1: E$12.7, E$14.1, E$15.2, E$16.1
- removed net S$14: E$1.10, E$16.2
- removed net S$23: E$14.2, E$3.4
- removed net S$24: E$1.23, E$1.24, E$10.1, E$10.7, E$12.1
- new net 5V: E$14.2, E$3.4, E$5.1
- new net GND: E$1.23, E$1.24, E$10.1, E$10.7, E$12.1, E$12.7, E$14.1, E$15.2, E$5.2
- new net LED: E$2.8
- new net VBAT: E$1.10
- net S$16: now also E$8.4
Routing:
- net GND: track 0.00 -> 410.1 mm, vias 0 -> 1
- net 5V: track 0.00 -> 175.5 mm
- net S$16: track 106.0 -> 237.6 mm
- net S$23: track 119.1 -> 0.00 mm
- net VBAT: track 0.00 -> 113.2 mm
- net S$24: track 86.0 -> 0.00 mm
- net LED: track 0.00 -> 65.2 mm, vias 0 -> 1
- net S$1: track 41.1 -> 0.00 mm
- net +12V: track 202.6 -> 205.4 mm
Changed lines of the file:
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@@
 <element name="E$3" library="pinhead" package="1X04" value="" x="5.08" y="34.29" rot="R180"/>
 <element name="E$4" library="con-wago-500" package="W237-4" value="" x="86.36" y="33.02" rot="R90"/>
-<element name="E$5" library="con-wago-500" package="W237-4" value="" x="81.28" y="78.74" rot="R180"/>
-<element name="E$6" library="con-wago-500" package="W237-4" value="" x="5.08" y="60.96" rot="R270"/>
 <element name="E$7" library="con-wago-500" package="W237-4" value="" x="86.36" y="7.62" rot="R90"/>
-<element name="E$8" library="con-wago-500" package="W237-4" value="" x="58.42" y="78.74" rot="R180"/>
+<element name="E$8" library="con-wago-500" package="W237-4" value="" x="43.18" y="78.105" rot="R180"/>
 <element name="E$9" library="pinhead" package="1X08" value="" x="55.88" y="12.7" rot="R90"/>
 <element name="E$10" library="pinhead" package="1X08" value="" x="68.58" y="12.7" rot="R90"/>
@@
 <element name="E$14" library="con-wago-500" package="W237-102" value="" x="86.36" y="50.8" rot="R90"/>
 <element name="E$13" library="con-wago-500" package="W237-103" value="" x="86.36" y="66.04" rot="R90"/>
-<element name="E$15" library="con-wago-500" package="W237-102" value="" x="5.08" y="78.74" rot="R270"/>
-<element name="E$16" library="con-wago-500" package="W237-102" value="" x="22.86" y="78.74" rot="R180"/>
+<element name="E$15" library="con-wago-500" package="W237-102" value="" x="4.445" y="78.105" rot="R270"/>
+<element name="E$16" library="con-wago-500" package="W237-102" value="" x="20.32" y="78.105" rot="R270"/>
+<element name="E$5" library="con-wago-500" package="W237-102" value="" x="86.36" y="78.105" rot="R180"/>
 </elements>
 <signals>
@@
 <wire x1="81.915" y1="41.91" x2="68.58" y2="41.91" width="1.4224" layer="1"/>
 </signal>
-<signal name="S$23">
+<signal name="5V">
 <contactref element="E$3" pad="4"/>
 <wire x1="1.27" y1="38.1" x2="1.27" y2="34.29" width="1.6764" layer="1"/>
@@
 <wire x1="85.09" y1="63.5" x2="74.93" y2="53.34" width="1.6764" layer="1"/>
 <wire x1="49.53" y1="53.34" x2="74.93" y2="53.34" width="1.6764" layer="1"/>
+<contactref element="E$5" pad="1"/>
+<wire x1="88.86" y1="79.375" x2="88.86" y2="76.24" width="1.6764" layer="1"/>
+<wire x1="88.86" y1="76.24" x2="88.9" y2="76.2" width="1.6764" layer="1"/>
+<wire x1="88.9" y1="76.2" x2="91.44" y2="73.66" width="1.6764" layer="1"/>
+<wire x1="91.44" y1="73.66" x2="91.44" y2="63.5" width="1.6764" layer="1"/>
+<wire x1="50.8" y1="79.375" x2="77.47" y2="79.375" width="1.6764" layer="1"/>
+<wire x1="77.47" y1="79.375" x2="80.645" y2="76.2" width="1.6764" layer="1"/>
+<wire x1="80.645" y1="76.2" x2="88.9" y2="76.2" width="1.6764" layer="1"/>
 </signal>
 <signal name="S$19">
@@
 <wire x1="88.265" y1="71.12" x2="87.65" y2="71.04" width="0" layer="19" extent="1-1"/>
 </signal>
-<signal name="S$14">
-<contactref element="E$16" pad="2"/>
+<signal name="VBAT">
 <contactref element="E$1" pad="10"/>
-<wire x1="21.59" y1="6.35" x2="20.36" y2="80.01" width="0" layer="19" extent="1-1"/>
-</signal>
-<signal name="S$15">
+<wire x1="21.59" y1="6.35" x2="21.59" y2="11.43" width="1.6764" layer="1"/>
+<wire x1="21.59" y1="11.43" x2="10.16" y2="22.86" width="1.6764" layer="1"/>
+<wire x1="10.16" y1="22.86" x2="-7.62" y2="22.86" width="1.6764" layer="1"/>
+<wire x1="-7.62" y1="22.86" x2="-7.62" y2="66.675" width="1.6764" layer="1"/>
+<wire x1="19.05" y1="75.565" x2="13.335" y2="75.565" width="1.6764" layer="1"/>
+<wire x1="13.335" y1="75.565" x2="5.08" y2="67.31" width="1.6764" layer="1"/>
+<wire x1="5.08" y1="67.31" x2="-6.985" y2="67.31" width="1.6764" layer="1"/>
+<wire x1="-6.985" y1="67.31" x2="-7.62" y2="66.675" width="1.6764" layer="1"/>
+</signal>
+<signal name="+12V">
 <contactref element="E$12" pad="8"/>
 <contactref element="E$15" pad="1"/>
@@
 <wire x1="91.44" y1="50.8" x2="91.44" y2="21.59" width="1.6764" layer="1"/>
 <wire x1="91.44" y1="21.59" x2="68.58" y2="21.59" width="1.6764" layer="1"/>
-<wire x1="3.81" y1="81.24" x2="3.81" y2="82.55" width="1.6764" layer="1"/>
-<wire x1="3.81" y1="82.55" x2="5.08" y2="83.82" width="1.6764" layer="1"/>
-<wire x1="5.08" y1="83.82" x2="91.44" y2="83.82" width="1.6764" layer="1"/>
-<wire x1="91.44" y1="83.82" x2="93.98" y2="81.28" width="1.6764" layer="1"/>
+<wire x1="3.175" y1="80.605" x2="3.81" y2="82.55" width="1.6764" layer="1"/>
+<wire x1="3.81" y1="82.55" x2="5.08" y2="85.09" width="1.6764" layer="1"/>
+<wire x1="5.08" y1="85.09" x2="91.44" y2="85.09" width="1.6764" layer="1"/>
+<wire x1="91.44" y1="85.09" x2="93.98" y2="81.28" width="1.6764" layer="1"/>
 <wire x1="93.98" y1="81.28" x2="93.98" y2="50.8" width="1.6764" layer="1"/>
 <wire x1="93.98" y1="50.8" x2="91.44" y2="50.8" width="1.6764" layer="1"/>
@@
 <wire x1="11.43" y1="3.81" x2="11.43" y2="6.35" width="1.6764" layer="1"/>
 <wire x1="68.58" y1="6.35" x2="62.865" y2="6.35" width="1.6764" layer="1"/>
-</signal>
-<signal name="S$1">
+<contactref element="E$8" pad="4"/>
+<wire x1="11.43" y1="6.35" x2="11.43" y2="17.78" width="1.6764" layer="1"/>
+<wire x1="11.43" y1="17.78" x2="9.525" y2="19.685" width="1.6764" layer="1"/>
+<wire x1="9.525" y1="19.685" x2="-8.89" y2="19.685" width="1.6764" layer="1"/>
+<wire x1="-8.89" y1="19.685" x2="-10.16" y2="20.955" width="1.6764" layer="1"/>
+<wire x1="-10.16" y1="20.955" x2="-10.16" y2="67.31" width="1.6764" layer="1"/>
+<wire x1="-10.16" y1="67.31" x2="-5.08" y2="72.39" width="1.6764" layer="1"/>
+<wire x1="-5.08" y1="72.39" x2="6.35" y2="72.39" width="1.6764" layer="1"/>
+<wire x1="6.35" y1="72.39" x2="12.065" y2="78.105" width="1.6764" layer="1"/>
+<wire x1="12.065" y1="78.105" x2="34.41" y2="78.105" width="1.6764" layer="1"/>
+<wire x1="34.41" y1="78.105" x2="35.68" y2="79.375" width="1.6764" layer="1"/>
+</signal>
+<signal name="GND">
+<contactref element="E$15" pad="2"/>
+<wire x1="3.175" y1="75.605" x2="5.755" y2="76.24" width="1.6764" layer="1"/>
+<wire x1="5.755" y1="76.24" x2="12.065" y2="82.55" width="1.6764" layer="1"/>
+<wire x1="12.065" y1="82.55" x2="19.05" y2="82.55" width="1.6764" layer="1"/>
+<wire x1="19.05" y1="82.55" x2="25.4" y2="82.55" width="1.6764" layer="1"/>
+<wire x1="19.05" y1="80.645" x2="19.05" y2="82.55" width="1.6764" layer="1"/>
 <contactref element="E$14" pad="1"/>
 <wire x1="88.9" y1="48.26" x2="87.67" y2="48.26" width="1.6764" layer="1"/>
@@
 <contactref element="E$12" pad="7"/>
 <wire x1="68.58" y1="44.45" x2="78.74" y2="44.45" width="1.6764" layer="1"/>
-<contactref element="E$16" pad="1"/>
-<wire x1="25.36" y1="80.01" x2="68.58" y2="44.45" width="0" layer="19" extent="1-1"/>
-<contactref element="E$15" pad="2"/>
-<wire x1="3.81" y1="76.24" x2="25.36" y2="80.01" width="0" layer="19" extent="1-1"/>
-<wire x1="-2.58" y1="76.24" x2="3.81" y2="76.24" width="1.4224" layer="1"/>
-<wire x1="-2.54" y1="63.5" x2="-2.58" y2="76.24" width="1.4224" layer="1"/>
-</signal>
-<signal name="S$24">
+<contactref element="E$5" pad="2"/>
+<wire x1="83.86" y1="79.375" x2="83.82" y2="79.375" width="1.6764" layer="1"/>
+<wire x1="83.82" y1="79.375" x2="80.645" y2="82.55" width="1.6764" layer="1"/>
+<wire x1="80.645" y1="82.55" x2="40.64" y2="82.55" width="1.6764" layer="1"/>
+<wire x1="40.64" y1="82.55" x2="25.4" y2="82.55" width="1.6764" layer="1"/>
+<wire x1="68.58" y1="44.45" x2="67.31" y2="44.45" width="1.6764" layer="16"/>
+<wire x1="67.31" y1="44.45" x2="65.405" y2="42.545" width="1.6764" layer="16"/>
+<wire x1="65.405" y1="42.545" x2="65.405" y2="30.48" width="1.6764" layer="16"/>
+<wire x1="65.405" y1="30.48" x2="66.675" y2="29.21" width="1.6764" layer="16"/>
+<wire x1="66.675" y1="29.21" x2="68.58" y2="29.21" width="1.6764" layer="16"/>
+<wire x1="40.64" y1="79.375" x2="40.64" y2="82.55" width="1.6764" layer="1"/>
 <contactref element="E$10" pad="7"/>
 <contactref element="E$12" pad="1"/>
@@
 <wire x1="65.405" y1="28.575" x2="66.675" y2="29.21" width="1.27" layer="1"/>
 <wire x1="66.675" y1="29.21" x2="68.58" y2="29.21" width="1.27" layer="1"/>
-<wire x1="39.37" y1="6.35" x2="65.405" y2="19.05" width="0" layer="19" extent="1-1"/>
-<wire x1="39.37" y1="3.81" x2="39.37" y2="6.35" width="0" layer="19" extent="1-1"/>
+<wire x1="68.58" y1="3.81" x2="68.58" y2="-5.08" width="1.6764" layer="1"/>
+<wire x1="68.58" y1="-5.08" x2="39.37" y2="-5.08" width="1.6764" layer="1"/>
+<via x="39.37" y="-5.08" extent="1-16" drill="1.2" shape="square"/>
+<wire x1="39.37" y1="6.35" x2="39.37" y2="3.81" width="1.6764" layer="16"/>
+<wire x1="39.37" y1="6.35" x2="39.37" y2="-5.08" width="1.6764" layer="16"/>
+<wire x1="39.37" y1="-5.08" x2="-2.54" y2="-5.08" width="1.6764" layer="1"/>
+<wire x1="-2.54" y1="-5.08" x2="-12.7" y2="0" width="1.6764" layer="1"/>
+<wire x1="-12.7" y1="0" x2="-12.7" y2="68.58" width="1.6764" layer="1"/>
+<wire x1="3.175" y1="75.565" x2="-5.715" y2="75.565" width="1.6764" layer="1"/>
+<wire x1="-5.715" y1="75.565" x2="-12.7" y2="68.58" width="1.6764" layer="1"/>
+<wire x1="3.175" y1="75.565" x2="3.175" y2="75.605" width="0" layer="19" extent="1-1"/>
 </signal>
 <signal name="S$10">
@@
 <wire x1="43.18" y1="30.48" x2="43.18" y2="36.83" width="0.8128" layer="1"/>
 </signal>
+<signal name="LED">
+<contactref element="E$2" pad="8"/>
+<wire x1="19.05" y1="34.29" x2="19.05" y2="50.8" width="1.6764" layer="16"/>
+<via x="19.05" y="50.8" extent="1-16" drill="1.2" shape="square"/>
+<wire x1="19.05" y1="50.8" x2="23.495" y2="50.8" width="1.6764" layer="1"/>
+<wire x1="23.495" y1="50.8" x2="26.67" y2="53.975" width="1.6764" layer="1"/>
+<wire x1="26.67" y1="53.975" x2="38.735" y2="53.975" width="1.6764" layer="1"/>
+<wire x1="38.735" y1="53.975" x2="45.72" y2="60.96" width="1.6764" layer="1"/>
+<wire x1="45.72" y1="78.74" x2="45.72" y2="60.96" width="1.6764" layer="1"/>
+</signal>
 </signals>

Commit message: modified:   .gitignore 	modified:   pcb/projekt.brd 	modified:   pcb/readme.scr
Parts:
- added E$17: (no value), con-wago-500:W237-4
- added E$6: (no value), 40xx:SO16
- moved E$8 1.91 mm to (43.2, 76.2)
Connections:
- removed net S$16: E$1.1, E$1.2, E$10.2, E$12.2, E$8.4
- new net S$1: E$2.11, E$6.13, E$6.14
- new net S$14: E$17.1, E$6.1, E$6.2
- new net S$15: E$17.2, E$6.3, E$6.4
- new net S$25: E$1.1, E$1.2, E$10.2, E$12.2
- net +12V: now also E$17.3, E$17.4, E$6.9
- net GND: now also E$6.8, E$8.3
- net LED: now also E$6.15, E$6.16, E$8.2
Routing:
- net S$25: track 0.00 -> 250.8 mm
- net S$16: track 237.6 -> 0.00 mm
- net S$1: track 0.00 -> 189.3 mm
- net GND: track 410.1 -> 494.9 mm
- net +12V: track 205.4 -> 264.9 mm, vias 0 -> 1
- net LED: track 65.2 -> 94.0 mm
- net S$14: track 0.00 -> 11.4 mm
- net VBAT: track 113.2 -> 123.2 mm
- net S$15: track 0.00 -> 6.45 mm
- net 5V: track 175.5 -> 180.4 mm
- net S$23: track 0.00 -> 1.80 mm
- net S$13: track 154.7 -> 153.5 mm
