File: pcb/projekt.brd (EAGLE design)
At the start: 17 parts

Commit message: 'board'
Parts:
- added E$18, E$19: (no value), wirepad:3,17/1,2
Connections:
- new net S$26: E$18.1, E$8.1
Routing:
- net S$28: track 0.00 -> 30.4 mm, vias 0 -> 1
- net S$26: track 0.00 -> 27.9 mm
- net S$27: track 0.00 -> 21.4 mm, vias 0 -> 1
- net GND: track 494.9 -> 506.7 mm
- net S$16: track 0.00 -> 4.34 mm
Changed lines of the file:
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@@
 <layer number="21" name="tPlace" color="7" fill="1" visible="yes" active="yes"/>
 <layer number="22" name="bPlace" color="7" fill="1" visible="yes" active="yes"/>
-<layer number="23" name="tOrigins" color="15" fill="1" visible="no" active="yes"/>
-<layer number="24" name="bOrigins" color="15" fill="1" visible="no" active="yes"/>
-<layer number="25" name="tNames" color="7" fill="1" visible="no" active="yes"/>
-<layer number="26" name="bNames" color="7" fill="1" visible="no" active="yes"/>
-<layer number="27" name="tValues" color="7" fill="1" visible="no" active="yes"/>
-<layer number="28" name="bValues" color="7" fill="1" visible="no" active="yes"/>
+<layer number="23" name="tOrigins" color="15" fill="1" visible="yes" active="yes"/>
+<layer number="24" name="bOrigins" color="15" fill="1" visible="yes" active="yes"/>
+<layer number="25" name="tNames" color="7" fill="1" visible="yes" active="yes"/>
+<layer number="26" name="bNames" color="7" fill="1" visible="yes" active="yes"/>
+<layer number="27" name="tValues" color="7" fill="1" visible="yes" active="yes"/>
+<layer number="28" name="bValues" color="7" fill="1" visible="yes" active="yes"/>
 <layer number="29" name="tStop" color="7" fill="3" visible="no" active="yes"/>
 <layer number="30" name="bStop" color="7" fill="6" visible="no" active="yes"/>
@@
 <circle x="19.05" y="31.75" radius="0.898025" width="0.4064" layer="1"/>
 <circle x="1.27" y="34.29" radius="0.898025" width="0.4064" layer="1"/>
-<dimension x1="-5.08" y1="114.3" x2="34.925" y2="114.3" x3="14.9225" y3="116.84" textsize="1.778" layer="16"/>
-<dimension x1="-5.08" y1="114.3" x2="-5.08" y2="96.52" x3="-7.62" y3="105.41" textsize="1.778" layer="16"/>
-<rectangle x1="-5.08" y1="52.07" x2="34.925" y2="69.85" layer="16" rot="R18"/>
 <circle x="-6.985" y="63.5" radius="1.27" width="1.6764" layer="1"/>
 <circle x="-1.27" y="46.99" radius="1.27" width="1.6764" layer="1"/>
 <circle x="31.115" y="75.565" radius="1.27" width="1.6764" layer="1"/>
 <circle x="36.195" y="59.055" radius="1.27" width="1.6764" layer="1"/>
+<dimension x1="-19.685" y1="-10.795" x2="94.615" y2="-10.16" x3="37.535334375" y3="-23.138303125" textsize="1.778" layer="16"/>
+<dimension x1="101.6" y1="88.265" x2="101.6" y2="-11.43" x3="128.905" y3="38.4175" textsize="1.778" layer="16" dtype="horizontal"/>
 </plain>
 <attributes>
@@
 <element name="E$6" library="40xx" package="SO16" value="" x="66.04" y="68.58" rot="R180"/>
 <element name="E$17" library="con-wago-500" package="W237-4" value="" x="66.04" y="76.2" rot="R180"/>
+<element name="E$18" library="wirepad" package="3,17/1,2" value="" x="31.115" y="75.565"/>
+<element name="E$19" library="wirepad" package="3,17/1,2" value="" x="36.195" y="59.055"/>
 </elements>
 <signals>
@@
 <wire x1="71.12" y1="68.58" x2="73.025" y2="66.675" width="0.8128" layer="1"/>
 <wire x1="73.025" y1="66.675" x2="73.025" y2="65.405" width="0.8128" layer="1"/>
-<via x="73.025" y="65.405" extent="1-16" drill="1.2" shape="square"/>
+<via x="73.025" y="65.405" extent="1-16" drill="0.5" shape="square"/>
 <wire x1="73.025" y1="65.405" x2="73.025" y2="51.435" width="0.8128" layer="16"/>
 <wire x1="73.025" y1="51.435" x2="68.58" y2="46.99" width="0.8128" layer="16"/>
@@
 <wire x1="-5.08" y1="-5.08" x2="-17.78" y2="7.62" width="1.6764" layer="1"/>
 <wire x1="-17.78" y1="7.62" x2="-17.78" y2="66.04" width="1.6764" layer="1"/>
-<wire x1="3.175" y1="75.565" x2="-8.255" y2="75.565" width="1.6764" layer="1"/>
+<wire x1="3.175" y1="75.565" x2="1.27" y2="75.565" width="1.6764" layer="1"/>
+<wire x1="1.27" y1="75.565" x2="-8.255" y2="75.565" width="1.6764" layer="1"/>
 <wire x1="-8.255" y1="75.565" x2="-17.78" y2="66.04" width="1.6764" layer="1"/>
 <contactref element="E$6" pad="8"/>
@@
 <wire x1="36.83" y1="58.42" x2="36.83" y2="60.96" width="1.6764" layer="1"/>
 <wire x1="36.83" y1="60.96" x2="40.64" y2="64.77" width="1.6764" layer="1"/>
-<wire x1="40.64" y1="64.77" x2="40.64" y2="81.28" width="1.6764" layer="1"/>
+<wire x1="40.64" y1="64.77" x2="40.64" y2="74.93" width="1.6764" layer="1"/>
+<wire x1="40.64" y1="74.93" x2="40.64" y2="80.01" width="1.6764" layer="1"/>
+<wire x1="40.64" y1="80.01" x2="40.64" y2="81.28" width="1.6764" layer="1"/>
 <wire x1="3.175" y1="75.565" x2="3.175" y2="75.605" width="0" layer="19" extent="1-1"/>
+<wire x1="1.27" y1="75.565" x2="1.27" y2="76.2" width="1.6764" layer="1"/>
+<wire x1="1.27" y1="76.2" x2="1.905" y2="76.835" width="1.6764" layer="1"/>
+<wire x1="1.905" y1="76.835" x2="5.08" y2="76.835" width="1.6764" layer="1"/>
+<wire x1="5.08" y1="76.835" x2="5.715" y2="76.2" width="1.6764" layer="1"/>
+<wire x1="40.64" y1="74.93" x2="39.37" y2="76.2" width="1.6764" layer="1"/>
+<wire x1="39.37" y1="76.2" x2="39.37" y2="78.74" width="1.6764" layer="1"/>
+<wire x1="39.37" y1="78.74" x2="40.64" y2="80.01" width="1.6764" layer="1"/>
 </signal>
 <signal name="S$10">
@@
 </signal>
 <signal name="S$24">
-<via x="73.025" y="65.405" extent="1-16" drill="1.2" shape="square"/>
+<via x="73.025" y="65.405" extent="1-16" drill="0.8" shape="square"/>
 </signal>
 <signal name="S$1">
@@
 <wire x1="21.59" y1="78.105" x2="12.065" y2="78.105" width="1.6764" layer="1"/>
 </signal>
+<signal name="S$16">
+<wire x1="37.465" y1="-5.715" x2="38.1" y2="-6.35" width="1.6764" layer="1"/>
+<wire x1="38.1" y1="-6.35" x2="40.64" y2="-6.35" width="1.6764" layer="1"/>
+<wire x1="40.64" y1="-6.35" x2="41.275" y2="-5.715" width="1.6764" layer="1"/>
+</signal>
+<signal name="S$26">
+<contactref element="E$8" pad="1"/>
+<contactref element="E$18" pad="1"/>
+<wire x1="31.115" y1="75.565" x2="31.115" y2="73.025" width="1.6764" layer="16"/>
+<wire x1="31.115" y1="73.025" x2="33.02" y2="71.12" width="1.6764" layer="16"/>
+<wire x1="33.02" y1="71.12" x2="48.26" y2="71.12" width="1.6764" layer="16"/>
+<wire x1="48.26" y1="71.12" x2="50.8" y2="73.66" width="1.6764" layer="16"/>
+<wire x1="50.8" y1="73.66" x2="50.8" y2="77.35" width="1.6764" layer="16"/>
+<wire x1="50.8" y1="77.35" x2="50.68" y2="77.47" width="1.6764" layer="16"/>
+</signal>
+<signal name="S$27">
+<via x="-6.985" y="63.5" extent="1-16" drill="1.6" shape="square"/>
+<wire x1="-6.985" y1="63.5" x2="-6.985" y2="70.485" width="1.6764" layer="16"/>
+<wire x1="-6.985" y1="70.485" x2="3.175" y2="80.645" width="1.6764" layer="16"/>
+</signal>
+<signal name="S$28">
+<via x="-1.27" y="46.99" extent="1-16" drill="1.6" shape="square"/>
+<wire x1="-1.27" y1="46.99" x2="-1.27" y2="71.12" width="1.6764" layer="16"/>
+<wire x1="-1.27" y1="71.12" x2="3.175" y2="75.565" width="1.6764" layer="16"/>
+</signal>
 </signals>
